File: KiCad_Schematics/PowerDistribution/PowerDistribution.sch (KiCad schematic (older format))
At the start: 20 parts, among them K1 HE1AN-S-DC12V, K2 HE1AN-S-DC12V, M1 T200_Thruster, M2 T200_Thruster, SW1 ChangeoverSwitch, SW2 SW_SPST, U1 FuseBlock, U2 FuseBlock

Commit message: updated schematics
Parts:
- removed CB1, CB2: CircuitBreaker_30A, symbol Device:CircuitBreaker_1P_US
- removed F2: 10A, symbol Device:Fuse
- removed K1, K2: HE1AN-S-DC12V, Relay_THT:Relay_StandexMeder_DIP_LowProfile, symbol Relay:DIPxx-1Axx-11x
- removed M1, M2: T200_Thruster, symbol Motor:Motor_DC
- removed V1: 22.2, symbol pspice:VSOURCE
- removed V2: 12, symbol pspice:VSOURCE
- removed V3: 11.1, symbol pspice:VSOURCE
- added F6: 4A, symbol Device:Fuse
- F1: renamed from F6; value 7.5A -> 3A
- F3: renamed from F8; value 3A -> 5A
- F5: renamed from F4; value 3A -> 7.5A
- F7: renamed from F3; value 3A -> 2A
- SW2: value SW_SPST -> MotorDisconnect
- renumbered F7 to F2, F1 to F4, U2 to U1, U1 to U2
Connections:
- net labels added: +11.1V_Battery, +14.8V_Battery, +22.2V_Battery, +BATT_14.8V, -11.1V_Battery, -14.8V_Battery, -22.2V_Battery, -V_LEFT_ESC, -V_RIGHT_ESC, 11.1V-OFF-12V, 12V_Shore, 22.2V-OFF-12V, E-Receiver, E-Receiver_GND, FeatherUSB, FeatherUSB_GND, GL-iNet, GL-iNet_GND, GND-OFF-GND, RPi4, RPi4_GND, TP-Link, TP-Link_GND, USBHub, USBHub_GND
- net labels removed: 0, 11.1V, 12V, 14.8V, 22.2V, EmergencyRelayController, EmergencyRelayController_GND, FeatherPower, FeatherPower_GND, MotorRelay, MotorRelay_GND, Network, Network_GND, RPi, RPi_GND, StatusLights, StatusLights_GND, USB_Hub, USB_Hub_GND
- wire segments 88 -> 70
- no-connect marks 16 -> 21
Other:
- note added: "Going to Emergency \nStop Relays"
- note removed: "Simulated Sources\n"
- moved on the sheet: F1, F2, F3, F4, F5, F7, SW1, U1, U2

Commit message: Updates to images, schematics, and arduino code
Parts:
- added CB1, CB2: 30A, symbol Device:CircuitBreaker_1P_US
- added SW1: ShorePowerEnable, symbol Switch:SW_SPST
- renumbered SW1 to SW2, SW2 to SW3
Connections:
- net -14.8V_Battery: now also CB1.2, CB2.2
- net at U1.~: now also F3.2
- net at U2.~: now also F6.2
- new net -V_LEFT_ESC: CB2.1
- new net -V_RIGHT_ESC: CB1.1
- new net 5V_Shore: SW1.1 (A)
- new net Enable_Shore: SW1.2 (B)
Other:
- note added: "SW1 Turns on/off the \nshore power supply"
- note added: "To Emergency \nStop Relays"
- note removed: "Going to Emergency \nStop Relays"
- moved on the sheet: F1, F2, F3, F4, F5, F6, F7, SW2, SW3, U1, U2
