File: KiCad_Schematics/TeensySchematic/TeensySchematic.sch (KiCad schematic (older format))
At the start: 5 parts, among them J1 LEFT_ESC, J2 RIGHT_ESC, U1 Teensy3.2, U2 BNO055, U3 Adafruit_Ultimate_GPS

Commit message: updated schematics
Parts:
- U1: symbol TeensySchematic-rescue:Teensy3.2-Teensy -> TeensySchematic-rescue:Teensy3.2-Teensy-TeensySchematic-rescue
- U2: symbol TeensySchematic-rescue:BNO055-AdafruitBoards -> TeensySchematic-rescue:BNO055-AdafruitBoards-TeensySchematic-rescue
- U3: symbol MCU_Module:Adafruit_Ultimate_GPS -> TeensySchematic-rescue:Adafruit_Ultimate_GPS-MCU_Module
Changed lines of the file:
@@
 Sheet 1 1
 Title "Teensy Motor Control, GPS, and IMU Board"
-Date "2020-01-31"
-Rev "1"
+Date "2020-04-23"
+Rev "2"
 Comp "Temple University College of Engineering"
 Comment1 "Author: Byron Gaspard"
 Comment2 "Senior Design Project II"
-Comment3 "RoboBoat - TeamB04"
+Comment3 "RoboBoat - Team B04"
 Comment4 ""
 $EndDescr
 $Comp
-L TeensySchematic-rescue:BNO055-AdafruitBoards U2
+L TeensySchematic-rescue:BNO055-AdafruitBoards-TeensySchematic-rescue U2
 U 1 1 5E279D74
 P 8200 3900
@@
 $EndComp
 $Comp
-L MCU_Module:Adafruit_Ultimate_GPS U3
+L TeensySchematic-rescue:Adafruit_Ultimate_GPS-MCU_Module U3
 U 1 1 5E2C4F7F
 P 3450 4900
@@
 $EndComp
 $Comp
-L TeensySchematic-rescue:Teensy3.2-Teensy U1
+L TeensySchematic-rescue:Teensy3.2-Teensy-TeensySchematic-rescue U1
 U 1 1 5E27E1D1
 P 6300 3250

Commit message: Updates to images, schematics, and arduino code
Other:
- note added: "Absolute Orientation IMU"
- note added: "GPS Module"
- note added: "PWM Output for Motor ESCs"
- note added: "Teensy Microcontroller"
- moved on the sheet: U2, U3
